File: Line-following-learn-to-solder-kit.kicad_sch (KiCad schematic)
At the start: 27 parts, among them M1 DC TTMOTOR 3-6V, M2 DC TTMOTOR 3-6V, Q1 S8550, Q2 S8550, SW1 SW_DPDT, U1 LM393

Commit message: v0.0 release. Still missing some 3d models, exact part number associations.
Parts:
- added H1: MountingHole for M5 skid foot, MountingHole:MountingHole_5mm_Pad_TopBottom, symbol Mechanical:MountingHole
- added H2: MountingHole for wires, LineFollowingRobotFootPrints:MountingHole_3mm, symbol Mechanical:MountingHole
- M2: footprint LineFollowingRobotFootPrints:TT-Motor -> LineFollowingRobotFootPrints:TT-Motor-mirrored
- Q1, Q2: footprint Package_TO_SOT_THT:TO-92_HandSolder -> LineFollowingRobotFootPrints:TO-92_HandSolder
- R1, R2: footprint Potentiometer_THT:Potentiometer_Runtron_RM-065_Vertical -> LineFollowingRobotFootPrints:Potentiometer_Runtron_RM-065_Vertical_hand_soldering
- R10, R11, R12, R3, R4, R5, R6, R7, R8, R9: footprint Resistor_THT:R_Axial_DIN0207_L6.3mm_D2.5mm_P7.62mm_Horizontal -> LineFollowingRobotFootPrints:R_Axial_DIN0207_L6.3mm_D2.5mm_P7.62mm_Horizontal_hand_soldering
- R13, R14: value LDR07 -> LDR; footprint OptoDevice:R_LDR_5.1x4.3mm_P3.4mm_Vertical -> LineFollowingRobotFootPrints:R_LDR_5.1x4.3mm_P3.4mm_Vertical_hand_soldering
- SW1: footprint (none) -> LineFollowingRobotFootPrints:MHPS2283
- U1: footprint (none) -> Package_DIP:DIP-8_W7.62mm_Socket_LongPads
- renumbered D3 to D5
Connections:
- net at BT1.1 (+), Q1.1 (E), Q2.1 (E)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: now also R2.3, R4.1, R5.2, R6.2; no longer R2.1, R4.2, R5.1, R6.1
- net at BT1.2 (-): now also SW1.3 (C); no longer SW1.2 (B)
- net at R8.1, U1.2 (-), U1.5 (+): now also R2.1; no longer R2.3
- net at Q2.2 (B), R10.2: now also R4.2; no longer R4.1
- net at C1.2, C2.2, D1.1 (K)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: now also M1.1 (+), M2.1 (+), SW1.2 (B); no longer M1.2 (-), M2.2 (-), SW1.1 (A)
- net at Q2.3 (C), R12.1: now also M1.2 (-); no longer M2.1 (+)
- net at R9.1: now also Q1.2 (B), R3.1; no longer U1.1
- net at C2.1, D5.2 (A): now also R6.1; no longer R6.2
- net at C1.1, D4.2 (A): now also R5.1; no longer R5.2
- net at Q1.3 (C), R11.1: now also M2.2 (-); no longer M1.1 (+)
- new net: R9.2, U1.1
- no-connect marks 4 -> 0
Other:
- company: (none) -> Team 3140 Flagship Robotics
- title: (none) -> Line Following Bot
- moved on the sheet: D1, M1, M2, R11, R12, R4, R5, R9, SW1
